File: pcb-chocmini/pcb-chocmini.kicad_pcb (KiCad board)
At the start: 2 copper layers, 132.6 x 63.9 mm, 42 parts, among them J1 OLED, SW00 SW_PUSH_LED, SW01 SW_PUSH_LED, SW02 SW_PUSH_LED, SW03 SW_PUSH_LED, SW04 SW_PUSH_LED, SW10 SW_PUSH_LED, SW11 SW_PUSH_LED, SW12 SW_PUSH_LED, SW13 SW_PUSH_LED, SW14 SW_PUSH_LED, SW20 SW_PUSH_LED, SW21 SW_PUSH_LED, SW22 SW_PUSH_LED, SW23 SW_PUSH_LED, SW24 SW_PUSH_LED, SW34 SW_PUSH_LED, U1 ProMicro

Commit message: updates
Parts:
- EN1: footprint Keebio-Parts:RotaryEncoder_EC11 -> Keebio-Parts:RotaryEncoder_EC11_Nonplated
Routing:
- net VDD: track 0.00 -> 418.8 mm, vias 0 -> 27
- net Col0: track 0.00 -> 173.1 mm
- net Col1: track 0.00 -> 148.3 mm
- net Row2: track 0.00 -> 133.3 mm, vias 0 -> 1
- net LED: track 0.00 -> 130.0 mm, vias 0 -> 1
- net Col2: track 0.00 -> 121.5 mm
- net Row0: track 0.00 -> 116.7 mm, vias 0 -> 2
- net Row1: track 0.00 -> 116.4 mm, vias 0 -> 1
- net Col3: track 0.00 -> 96.6 mm
- net Col4: track 0.00 -> 85.9 mm
- net Row3: track 0.00 -> 44.4 mm
- net ENB: track 0.00 -> 41.8 mm
- net ENA: track 0.00 -> 34.7 mm
- net Net-(SW14-Pad2): track 0.00 -> 32.5 mm, vias 0 -> 2
- net Net-(SW12-Pad2): track 0.00 -> 32.5 mm, vias 0 -> 2
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Other:
- board text added: "Rev 3 by dcpedit: github.com/dcpedit/artpad"
- board text removed: "Rev 1 by dcpedit: github.com/dcpedit/artpad"
